Commit message: feat: finish liosam sim

File: scout_gazebo/urdf/base.xacro (robot description, xacro)
@@ -1,7 +1,7 @@
 <?xml version="1.0"?>
-<robot name="scout_v2"  xmlns:xacro="http://ros.org/wiki/xacro">
+<robot name="scout_v2" xmlns:xacro="http://ros.org/wiki/xacro">
     <xacro:arg name="robot_namespace" default="/" />
     <!-- 属性封装 -->
-    <xacro:property name="M_PI" value="3.14159"/>
+    <xacro:property name="M_PI" value="3.14159" />
     <xacro:property name="base_x_size" value="0.9250000" />
     <xacro:property name="base_y_size" value="0.380000" />
@@ -12,7 +12,7 @@
     <xacro:property name="wheel_length" value="1.1653e-01" />
     <xacro:property name="wheel_radius" value="1.6459e-01" />
-    <xacro:arg name="gpu" default="true"/>
+    <xacro:arg name="gpu" default="true" />
     <xacro:property name="gpu" value="$(arg gpu)" />
-    <xacro:arg name="organize_cloud" default="true"/>
+    <xacro:arg name="organize_cloud" default="true" />
     <xacro:property name="organize_cloud" value="$(arg organize_cloud)" />
     <material name="black">
@@ -26,18 +26,20 @@
     <!-- <xacro:include filename="$(find scout_gazebo)/urdf/sensor_camera.xacro" /> -->
     <!-- D435i RGB-D相机相关 -->
-    <xacro:include filename="$(find realsense_ros_gazebo)/xacro/depthcam.xacro"/>
+    <!-- <xacro:include filename="$(find realsense_ros_gazebo)/xacro/depthcam.xacro" />
     <xacro:realsense_d435 sensor_name="camera" parent_link="base_link" rate="30.0">
-    <origin rpy="0 0 0" xyz="0 0 0.3"/>
-    </xacro:realsense_d435>
+        <origin rpy="0 0 0" xyz="0 0 0.3" />
+    </xacro:realsense_d435> -->
     <!-- VLP16 激光雷达 -->
     <xacro:include filename="$(find scout_gazebo)/urdf/laser_support.xacro" />
-    <xacro:include filename="$(find velodyne_description)/urdf/VLP-16.urdf.xacro"/>
-    <xacro:VLP-16 parent="support" name="velodyne" topic="/velodyne_points" organize_cloud="${organize_cloud}" hz="10" samples="440" gpu="${gpu}">
-          <origin xyz="0 0 ${support_length/2}" rpy="0 0 0" />
+    <xacro:include filename="$(find velodyne_description)/urdf/VLP-16.urdf.xacro" />
+    <xacro:VLP-16 parent="support" name="velodyne" topic="/velodyne_points"
+        organize_cloud="${organize_cloud}" hz="10" samples="1000" collision_range="0.3"
+        min_range="0.2" max_range="100.0" gpu="${gpu}">
+        <origin xyz="0 0 ${support_length/2}" rpy="0 0 0" />
     </xacro:VLP-16>
     <!-- IMU 模块 -->
-    <xacro:include filename="$(find scout_gazebo)/urdf/imu.xacro"/>
+    <xacro:include filename="$(find scout_gazebo)/urdf/imu.xacro" />
     <xacro:imu sensor_name="imu" parent_link="base_link">
-    <origin rpy="0 0 0" xyz="-0.03 0 ${base_z_size/2}"/>
+        <origin rpy="0 0 0" xyz="-0.03 0 ${base_z_size/2}" />
     </xacro:imu>
     <!-- 机器人导航控制模块 -->
@@ -48,5 +50,6 @@
             <origin xyz="0 0 0" rpy="0 0 0" />
             <geometry>
-                <!--<box size="${base_x_size} ${base_y_size} ${base_z_size}"/>-->
+                <!--<box
+                size="${base_x_size} ${base_y_size} ${base_z_size}"/>-->
                 <mesh filename="package://scout_gazebo/meshes/base_link.dae" />
             </geometry>
@@ -55,9 +58,9 @@
             <origin xyz="0 0 0.0008" rpy="0 0 0" />
             <geometry>
-                <box size="${base_x_size} ${base_y_size} ${base_z_size}"/>
+                <box size="${base_x_size} ${base_y_size} ${base_z_size}" />
             </geometry>
         </collision>
     </link>
-    <link name="base_footprint"/>
+    <link name="base_footprint" />
     <joint name="base_footprint_joint" type="fixed">
         <origin xyz="0 0 0" rpy="0 0 0" />
@@ -92,3 +95,15 @@
         <origin xyz="${-wheelbase/2} ${-track/2} ${wheel_vertical_offset}" rpy="3.14 0 0" />
     </xacro:scout_wheel_type2>
+    <gazebo>
+        <plugin name="p3d_base_controller" filename="libgazebo_ros_p3d.so">
+            <alwaysOn>true</alwaysOn>
+            <updateRate>100.0</updateRate>
+            <bodyName>base_link</bodyName>
+            <topicName>ground_truth/state</topicName>
+            <gaussianNoise>0.1</gaussianNoise>
+            <frameName>world</frameName>
+            <xyzOffsets>0 0 0</xyzOffsets>
+            <rpyOffsets>0 0 0</rpyOffsets>
+        </plugin>
+    </gazebo>
 </robot>

File: scout_gazebo/urdf/imu.xacro (robot description, xacro)
@@ -5,5 +5,5 @@
         <xacro:property name="imu_offset_y" value="0" />
         <xacro:property name="imu_offset_z" value="0.2" />
-        <xacro:property name="imu_size"     value="0.05" />
+        <xacro:property name="imu_size" value="0.05" />
         <xacro:property name="imu_m" value="0.01" /> <!-- imu质量 -->
         <!-- imu -->
@@ -11,6 +11,6 @@
             <!-- <origin xyz="${imu_offset_x} ${imu_offset_y} ${imu_offset_z}" rpy="0 0 0" /> -->
             <xacro:insert_block name="origin" />
-            <parent link="${parent_link}"/>
-            <child link="imu_base"/>
+            <parent link="${parent_link}" />
+            <child link="imu_base" />
         </joint>
         <link name="imu_base">
@@ -18,8 +18,8 @@
                 <origin rpy="0 0 0" xyz="0 0 0" />
                 <geometry>
-                        <box size="${imu_size} ${imu_size} ${imu_size}"/>
+                    <box size="${imu_size} ${imu_size} ${imu_size}" />
                 </geometry>
-                <material name= "black" >
-                <color rgba="1.0 0.0 0.0 0.6" />
+                <material name="black">
+                    <color rgba="1.0 0.0 0.0 0.6" />
                 </material>
             </visual>
@@ -30,5 +30,5 @@
                 <origin xyz="0.0 0.0 0" rpy="0.0 0.0 0.0" />
             </collision>
-            <xacro:Box_inertial_matrix m = "${imu_m}" l = "${imu_size}" w = "${imu_size}" h = "${imu_size}"/>
+            <xacro:Box_inertial_matrix m="${imu_m}" l="${imu_size}" w="${imu_size}" h="${imu_size}" />
         </link>
         <!-- 被引用的link -->
@@ -37,19 +37,21 @@
             <gravity>true</gravity>
             <sensor name="imu_sensor" type="imu">
-            <always_on>true</always_on>
-            <update_rate>100</update_rate>
-            <visualize>true</visualize>
-            <topic>__default_topic__</topic>
-            <plugin filename="libgazebo_ros_imu_sensor.so" name="imu_plugin">
-                <topicName>imu/data</topicName>
-                <bodyName>imu_base</bodyName>
-                <updateRateHZ>100.0</updateRateHZ>
-                <gaussianNoise>0.01</gaussianNoise>
-                <xyzOffset>0 0 0</xyzOffset>
-                <rpyOffset>0 0 0</rpyOffset>
-                <frameName>imu_base</frameName>
-            </plugin>
-            <pose>0 0 0 0 0 0</pose>
-        </sensor>
+                <always_on>true</always_on>
+                <!-- 传感器更新频率 -->
+                <update_rate>500</update_rate>
+                <visualize>true</visualize>
+                <topic>__default_topic__</topic>
+                <plugin filename="libgazebo_ros_imu_sensor.so" name="imu_plugin">
+                    <topicName>imu/data</topicName>
+                    <bodyName>imu_base</bodyName>
+                    <!-- 话题发布频率 -->
+                    <updateRateHZ>500.0</updateRateHZ>
+                    <gaussianNoise>0.01</gaussianNoise>
+                    <xyzOffset>0 0 0</xyzOffset>
+                    <rpyOffset>0 0 0</rpyOffset>
+                    <frameName>imu_base</frameName>
+                </plugin>
+                <pose>0 0 0 0 0 0</pose>
+            </sensor>
         </gazebo>
     </xacro:macro>
